Commit message: urdf changes

File: autocar_description/urdf/autocar edit.xacro (robot description, xacro)
@@ -17,5 +17,5 @@
   <joint name="hokuyo_joint" type="fixed">
     <axis xyz="0 1 0" />
-    <origin xyz="0 0 0.7" rpy="0 0 1.5708" />
+    <origin xyz="0 0.24 0" rpy="0 0 1.5708" />
     <parent link="chassis_link" />
     <child link="hokuyo_link" />
@@ -49,5 +49,5 @@
       <origin rpy="0 0 0" xyz="0 0 0" />
       <geometry>
-        <mesh filename="package://autocar_description/meshes/chassis_link.stl" scale="0.001 0.001 0.001" />
+        <box size="0.460 0.12 0.2" />
       </geometry>
       <material name="silver" />
@@ -56,25 +56,5 @@
       <origin rpy="0 0 0" xyz="0 0 0" />
       <geometry>
-        <mesh filename="package://autocar_description/meshes/chassis_link.stl" scale="0.001 0.001 0.001" />
-      </geometry>
-    </collision>
-  </link>
-  <joint name="spoiler_joint" type="fixed">
-    <origin xyz="0 0.05 -0.05" rpy="1.5708 0 3.14159" />
-    <parent link="chassis_link" />
-    <child link="spoiler_link" />
-  </joint>
-  <link name="spoiler_link">
-    <visual>
-      <origin rpy="0 0 0" xyz="0 0 0" />
-      <geometry>
-        <mesh filename="package://autocar_description/meshes/spoiler.stl" scale="0.001 0.001 0.001" />
-      </geometry>
-      <material name="silver" />
-    </visual>
-    <collision>
-      <origin rpy="0 0 0" xyz="0 0 0" />
-      <geometry>
-        <mesh filename="package://autocar_description/meshes/spoiler.stl" scale="0.001 0.001 0.001" />
+        <box size="0.460 0.12 0.2" />
       </geometry>
     </collision>
